File: STS1_EPS/STS1_EPS_PROTO_BCC_LTC4020/STS1_EPS_PROTO_BCC_LTC4020.sch (KiCad schematic (older format))
At the start: 17 parts, among them J1 1729267, J2 Output

Commit message: Intermediate state.
Parts:
- J1: footprint footprints:1729267 -> footprints:1984756
- J2: footprint footprints:1725656 -> footprints:1888807
Changed lines of the file:
@@
 F 0 "J2" H 10578 1453 60  0000 L CNN
 F 1 "Output" H 10578 1347 60  0000 L CNN
-F 2 "footprints:1725656" H 10450 1390 60  0001 C CNN
-F 3 "" H 10050 1450 60  0000 C CNN
+F 2 "footprints:1888807" H 10450 1390 60  0001 C CNN
+F 3 "https://www.mouser.at/datasheet/2/324/2/888807-1453113.pdf" H 10050 1450 60  0001 C CNN
 	1    10050 1450
 	1    0    0    -1
@@
 F 0 "J1" H 1742 1163 60  0000 C CNN
 F 1 "1729267" H 1742 1269 60  0000 C CNN
-F 2 "footprints:1729267" H 1900 2090 60  0001 C CNN
-F 3 "" H 1500 2950 60  0000 C CNN
+F 2 "footprints:1984756" H 1900 2090 60  0001 C CNN
+F 3 "https://www.mouser.at/datasheet/2/324/4/1984756-1458907.pdf" H 1500 2950 60  0001 C CNN
 	1    1500 2950
 	-1   0    0    1
