File: STS1_EPS/STS1_EPS_PROTO_BCC_LTC4020/template.sch (KiCad schematic (older format))
At the start: 13 parts, among them CON1 DISCO-CON1, CON11 DISCO-CON1, CON2 DISCO-CON2, CON21 DISCO-CON2, U4 coordinate_system

Commit message: Intermediate state.
Parts:
- added U5: logo, footprints:SpaceTeam_Logo, symbol STS-con:coordinate_system
Changed lines of the file:
@@
 Wire Wire Line
 	8200 5250 8200 5350
+$Comp
+L STS-con:coordinate_system U5
+U 1 1 60EF7724
+P 5300 1150
+F 0 "U5" H 5578 1221 50  0000 L CNN
+F 1 "logo" H 5578 1130 50  0000 L CNN
+F 2 "footprints:SpaceTeam_Logo" H 5300 1150 50  0001 C CNN
+F 3 "" H 5300 1150 50  0001 C CNN
+	1    5300 1150
+	1    0    0    -1
+$EndComp
 $EndSCHEMATC

Commit message: Intermediate state.
Parts:
- U5: footprint footprints:SpaceTeam_Logo -> footprints:STLogoTiny
Changed lines of the file:
@@
 $Descr A4 11693 8268
 encoding utf-8
-Sheet 4 4
+Sheet 5 5
 Title ""
 Date ""
@@
 F 0 "U5" H 5578 1221 50  0000 L CNN
 F 1 "logo" H 5578 1130 50  0000 L CNN
-F 2 "footprints:SpaceTeam_Logo" H 5300 1150 50  0001 C CNN
+F 2 "footprints:STLogoTiny" H 5300 1150 50  0001 C CNN
 F 3 "" H 5300 1150 50  0001 C CNN
 	1    5300 1150
