File: STS1_EPS/STS1_EPS_PROTO_BCC_LTC4020/STS1_EPS_BatteryCharger.sch (KiCad schematic (older format))
At the start: 32 parts, among them U1 LTC4020EUHF-PBF, U2 SI7272DP-T1-GE3, U3 SI7272DP-T1-GE3

Commit message: Reworked BCC
Parts:
- removed R2, R? (x6): R, symbol Device:R
- added C?: 200n, Capacitor_SMD:C_0805_2012Metric, symbol Device:C
- added C? (x2): 50µ, footprints:FE52N6J0506KB, symbol 2021-07-02_17-58-25:FE52N6J0506KB
- added C?: 2µ2, Capacitor_SMD:C_0805_2012Metric, symbol Device:C
- added C?: 10µ, Capacitor_SMD:C_0805_2012Metric, symbol Device:C
- added J4: External NTC, footprints:1725656, symbol Connector:Screw_Terminal_01x02
- added JP9, JP? (x4): Jumper_3_Open, Connector_PinHeader_2.54mm:PinHeader_1x03_P2.54mm_Vertical, symbol Jumper:Jumper_3_Open
- added R8: 200k, POT_TS53YL, symbol 2021-06-25_14-01-13:TS53YL_20K_20%
- added R9: 500k, Resistor_SMD:R_0805_2012Metric, symbol Device:R
- added R? (x2): 25k, Resistor_SMD:R_0805_2012Metric, symbol Device:R
- added R?: 44k, Resistor_SMD:R_0805_2012Metric, symbol Device:R
- added R?: 17k8, Resistor_SMD:R_0805_2012Metric, symbol Device:R
- added R? (x2): 100k, Resistor_SMD:R_0805_2012Metric, symbol Device:R
- added R?: 10m, footprints:CST0612-FC-R002E, symbol 2021-06-29_19-28-22:CST0612-FC-R002E
- added R?: 31k, Resistor_SMD:R_0805_2012Metric, symbol Device:R
- C4, C5: renamed from C?; value C -> 1µ; footprint (none) -> Capacitor_SMD:C_0805_2012Metric
- C6: renamed from C?; value C -> 100p; footprint (none) -> Capacitor_SMD:C_0805_2012Metric
- C7: renamed from C2; value C -> 200n; footprint (none) -> Capacitor_SMD:C_1812_4532Metric
- C8: renamed from C?; value C -> 330n; footprint (none) -> Capacitor_SMD:C_0805_2012Metric
- D1, D4: renamed from D?; footprint (none) -> LED_SMD:LED_0805_2012Metric
- D2, D3: renamed from D?; footprint (none) -> footprints:RB168MM-40TFTR
- J3: renamed from J?; footprint (none) -> footprints:1725656
- L1: footprint (none) -> Inductor_THT:L_Axial_L5.0mm_D3.6mm_P10.00mm_Horizontal_Murata_BL01RN1A2A2
- Q1: renamed from Q?; footprint TRANS_SI7135DP-T1-GE3 -> footprints:TRANS_SI7135DP-T1-GE3
- R1: renamed from R?; value R -> 28k; footprint (none) -> Resistor_SMD:R_0805_2012Metric
- R10: renamed from R?; value R -> 200k; footprint (none) -> Resistor_SMD:R_0805_2012Metric
- R11: renamed from R1; value R -> 5m; footprint (none) -> footprints:CST0612-FC-R002E; symbol Device:R -> 2021-06-29_19-28-22:CST0612-FC-R002E
- R12: renamed from R?; value R -> 5m; footprint (none) -> footprints:CST0612-FC-R002E; symbol Device:R -> 2021-06-29_19-28-22:CST0612-FC-R002E
- R14, R15: renamed from R?; value R -> 100; footprint (none) -> Resistor_SMD:R_0805_2012Metric
- R2: renamed from R?; value R -> 100k; footprint (none) -> Resistor_SMD:R_0805_2012Metric
- R3, R5: renamed from R?; value R -> 1k; footprint (none) -> Resistor_SMD:R_0805_2012Metric
- TH1: renamed from TH?; footprint (none) -> Resistor_SMD:R_0603_1608Metric
- U1: footprint LTC4020EUHF-PBF_ADI -> footprints:LTC4020EUHF-PBF
- U2, U3: footprint SON_DP-T1-GE3_VIS -> footprints:SI7272DP-T1-GE3
Connections:
- net SHDN is gone; now on net Vin: U1.9 (SHDN)
- net BAT: now also JP?.2 (C); no longer R1.2
- net CSP: now also R?.1, R?.1
- net FBG: now also R?.2, R?.2
- net GND: now also R12.3, R12.4, C?.1, C?.1, C?.2, C?.3, C?.3, C?.4, C?.4, J4.1 (Pin_1), JP?.3 (B), R9.1, R?.1, R?.1; no longer R12.2, U1.14 (TIMER)
- net ILIMIT: now also JP?.2 (C)
- net INTVCC: now also C?.2
- net SENSBOT: now also R12.2; no longer C7.2, R12.1, U3.1
- net SENSTOP: now also R11.4; no longer R11.2, U2.7, U2.8
- net VFB: now also R1.2, R?.2; no longer R1.1
- net VFBMAX: now also R?.1, R?.2; no longer U1.19 (VFBMIN)
- net Vin: now also R11.2, U1.28 (VC), R8.2, R8.3; no longer D1.2 (A), D4.2 (A)
- net Vout: now also D1.2 (A), D4.2 (A), R?.3, R?.4
- net VIN_REG: now reaches R10.1, U1.10 (VIN_REG)
- net VIN_REG: now also R8.1
- net RNGSS: now reaches U1.15 (RNG/SS)
- net RNGSS: now also JP?.2 (C)
- net at TH1.2: now also JP9.1 (A); no longer U1.16 (NTC)
- net RT: now reaches U1.8 (RT)
- net RT: now also R9.2
- net at Q1.1, R15.1: now also R?.1, R?.2
- new net: R11.3, U2.7, U2.8
- new net: C7.2, R12.1, U3.1
- new net: JP?.3 (B), R1.1
- new net: C?.1, JP?.1 (A)
- new net: J4.2 (Pin_2), JP9.3 (B)
- new net: C?.1, C?.2, JP?.3 (B) (x2)
- new net: JP?.1 (A), R?.2 (x2)
- new net: JP?.1 (A), R?.1
- new net NTC: JP9.2 (C), U1.16 (NTC)
- new net PVIN: C?.2
- new net TIMER: JP?.2 (C), U1.14 (TIMER)
- new net VFBMIN: R?.1, R?.2, U1.19 (VFBMIN)
Other:
- note added: "1s charging\nsoft start"
- note added: "3h charge \ntimer"
- note added: "External NTC"
- note added: "Li-Ion"
- note added: "LiFePo"
- note added: "No charge \ntimer"
- note added: "No charging\nsoft start"
- note added: "On-board NTC"
- moved on the sheet: C4, C5, C6, C7, C8, D1, D2, D3, D4, J3, L1, Q1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

Commit message: - STS1_EPS_PROTO_SCC_L6920 now uses the STS1 PCB template and is again ready for review. - WOrked on STS1_EPS_PROTO_BCC_LTC4020.
Parts:
- added C3: 680µ, Capacitor_Tantalum_SMD:CP_EIA-7361-438_AVX-U, symbol Device:CP
- added C9: 100n, Capacitor_SMD:C_0805_2012Metric, symbol Device:C
- added J10: BG2, Connector_PinHeader_2.54mm:PinHeader_1x01_P2.54mm_Vertical, symbol Connector:Conn_01x01_Male
- added J11: BGATE, Connector_PinHeader_2.54mm:PinHeader_1x01_P2.54mm_Vertical, symbol Connector:Conn_01x01_Male
- added J5: VIN_REG, Connector_PinHeader_2.54mm:PinHeader_1x01_P2.54mm_Vertical, symbol Connector:Conn_01x01_Male
- added J6: SHDN, Connector_PinHeader_2.54mm:PinHeader_1x01_P2.54mm_Vertical, symbol Connector:Conn_01x01_Male
- added J7: TG1, Connector_PinHeader_2.54mm:PinHeader_1x01_P2.54mm_Vertical, symbol Connector:Conn_01x01_Male
- added J8: TG2, Connector_PinHeader_2.54mm:PinHeader_1x01_P2.54mm_Vertical, symbol Connector:Conn_01x01_Male
- added J9: BG1, Connector_PinHeader_2.54mm:PinHeader_1x01_P2.54mm_Vertical, symbol Connector:Conn_01x01_Male
- added JP18: Top Side Current Shunt, Connector_PinHeader_2.54mm:PinHeader_1x02_P2.54mm_Vertical, symbol Device:Jumper_NC_Small
- added JP19: Low Side Current Shunt, Connector_PinHeader_2.54mm:PinHeader_1x02_P2.54mm_Vertical, symbol Device:Jumper_NC_Small
- added JP20: Battery Current, Connector_PinHeader_2.54mm:PinHeader_1x02_P2.54mm_Vertical, symbol Device:Jumper_NC_Small
- added R21: 600k, footprints:TS53YL 20K 20&percent_, symbol 2021-06-25_14-01-13:TS53YL_20K_20%
- added R22: 200k, Resistor_SMD:R_0805_2012Metric, symbol Device:R
- L1: value INDUCTOR -> 680n; footprint Inductor_THT:L_Axial_L5.0mm_D3.6mm_P10.00mm_Horizontal_Murata_BL01RN1A2A2 -> footprints:INDPM7366X500N
- R8: footprint POT_TS53YL -> footprints:TS53YL 20K 20&percent_
- gave numbers to parts that had none: 17
Connections:
- net BG1: now also J9.1 (Pin_1)
- net BG2: now also J10.1 (Pin_1)
- net BGATE: now also J11.1 (Pin_1)
- net GND: now also C3.2, C9.1, JP19.1, R22.2
- net SENSBOT: now also JP19.2
- net SENSTOP: now also JP18.1
- net TG1: now also J7.1 (Pin_1)
- net TG2: now also J8.1 (Pin_1)
- net VIN_REG: now also J5.1 (Pin_1)
- net Vin: now also C3.1, C9.2, R21.2, R21.3; no longer R11.2, U1.28 (VC), U1.7 (SENSVIN), U1.9 (SHDN)
- net Vout: no longer R14.1, R19.4
- net at Q1.1, R19.1: no longer R15.1, R19.2
- new net: JP20.2, R14.1, R19.4
- new net: JP20.1, R15.1, R19.2
- new net SENSVIN: JP18.2, R11.2, U1.7 (SENSVIN)
- new net SHDN: J6.1 (Pin_1), R21.1, R22.1, U1.9 (SHDN)
Other:
- moved on the sheet: C15, C7, C8, D1, D4, J4, JP13, JP9, Q1, R10, R14, R15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

Commit message: Intermediate state.
Parts:
- C11, C12: value 50µ -> 220µ; footprint footprints:FE52N6J0506KB -> Capacitor_Tantalum_SMD:CP_EIA-3528-12_Kemet-T; symbol 2021-07-02_17-58-25:FE52N6J0506KB -> Device:C
Connections:
- net GND: now also C11.1, C12.1; no longer C11.3, C11.4, C12.3, C12.4
- net ITH: now also U1.27 (ITH)
- net PVIN: now also U1.36 (PVIN)
- net VC: now also U1.28 (VC)
- net Vin: no longer U1.36 (PVIN)
- net at C11.2, JP10.3 (B): no longer C11.1
- net at C12.2, JP12.3 (B): no longer C12.1
Changed lines of the file:
@@
 $EndComp
 $Comp
-L 2021-07-02_17-58-25:FE52N6J0506KB C?
+L Device:C C?
 U 1 1 60F887F1
-P 900 4400
+P 850 4900
 AR Path="/60F887F1" Ref="C?"  Part="1"
 AR Path="/60B53241/60F887F1" Ref="C11"  Part="1"
-F 0 "C11" V 1347 4528 60  0000 L CNN
-F 1 "50µ" V 1453 4528 60  0000 L CNN
-F 2 "footprints:FE52N6J0506KB" H 1400 4540 60  0001 C CNN
-F 3 "" H 900 4400 60  0000 C CNN
-	1    900  4400
-	0    1    1    0
-$EndComp
-Wire Wire Line
-	850  4250 850  4400
-Wire Wire Line
-	850  4400 800  4400
-Wire Wire Line
-	900  4400 850  4400
-Connection ~ 850  4400
-Wire Wire Line
-	800  5400 850  5400
-Wire Wire Line
-	850  5500 850  5400
-Connection ~ 850  5400
-Wire Wire Line
-	850  5400 900  5400
+F 0 "C11" H 950 4800 60  0000 L CNN
+F 1 "220µ" H 950 5000 60  0000 L CNN
+F 2 "Capacitor_Tantalum_SMD:CP_EIA-3528-12_Kemet-T" H 1350 5040 60  0001 C CNN
+F 3 "https://www.mouser.at/datasheet/2/427/tmcu-1763538.pdf" H 850 4900 60  0001 C CNN
+	1    850  4900
+	-1   0    0    1
+$EndComp
 $Comp
 L Jumper:Jumper_3_Open JP10
@@
 U 1 1 60FC49BC
 P 1350 4900
-F 0 "R4" V 1143 4900 50  0000 C CNN
-F 1 "25k" V 1234 4900 50  0000 C CNN
+F 0 "R4" H 1200 4800 50  0000 C CNN
+F 1 "25k" H 1200 5000 50  0000 C CNN
 F 2 "Resistor_SMD:R_0805_2012Metric" V 1280 4900 50  0001 C CNN
 F 3 "~" H 1350 4900 50  0001 C CNN
@@
 $EndComp
 $Comp
-L 2021-07-02_17-58-25:FE52N6J0506KB C?
+L Device:C C?
 U 1 1 611C9576
-P 2200 4400
+P 2150 4900
 AR Path="/611C9576" Ref="C?"  Part="1"
 AR Path="/60B53241/611C9576" Ref="C12"  Part="1"
-F 0 "C12" V 2647 4528 60  0000 L CNN
-F 1 "50µ" V 2753 4528 60  0000 L CNN
-F 2 "footprints:FE52N6J0506KB" H 2700 4540 60  0001 C CNN
-F 3 "" H 2200 4400 60  0000 C CNN
-	1    2200 4400
-	0    1    1    0
-$EndComp
-Wire Wire Line
-	2150 4250 2150 4400
-Wire Wire Line
-	2150 4400 2100 4400
-Wire Wire Line
-	2200 4400 2150 4400
-Connection ~ 2150 4400
-Wire Wire Line
-	2100 5400 2150 5400
-Wire Wire Line
-	2150 5500 2150 5400
-Connection ~ 2150 5400
-Wire Wire Line
-	2150 5400 2200 5400
+F 0 "C12" H 2250 4800 60  0000 L CNN
+F 1 "220µ" H 2250 5050 60  0000 L CNN
+F 2 "Capacitor_Tantalum_SMD:CP_EIA-3528-12_Kemet-T" H 2650 5040 60  0001 C CNN
+F 3 "https://www.mouser.at/datasheet/2/427/tmcu-1763538.pdf" H 2000 6000 60  0001 C CNN
+	1    2150 4900
+	-1   0    0    1
+$EndComp
 $Comp
 L Jumper:Jumper_3_Open JP12
@@
 U 1 1 611C958B
 P 2650 4900
-F 0 "R7" V 2443 4900 50  0000 C CNN
-F 1 "25k" V 2534 4900 50  0000 C CNN
+F 0 "R7" H 2500 4800 50  0000 C CNN
+F 1 "25k" H 2500 5000 50  0000 C CNN
 F 2 "Resistor_SMD:R_0805_2012Metric" V 2580 4900 50  0001 C CNN
 F 3 "~" H 2650 4900 50  0001 C CNN
@@
 	1150 750  3150 750
 Text Label 4250 3350 2    50   ~ 0
-Vin
+PVIN
 Wire Wire Line
 	4550 3350 4250 3350
@@
 F 1 "680µ" H 3268 955 50  0000 L CNN
 F 2 "Capacitor_Tantalum_SMD:CP_EIA-7361-438_AVX-U" H 3188 850 50  0001 C CNN
-F 3 "https://www.mouser.at/datasheet/2/40/catalogue_TRM-1021477.pdf" H 3150 1000 50  0001 C CNN
+F 3 "https://www.mouser.at/datasheet/2/427/tmcu-1763538.pdf" H 3150 1000 50  0001 C CNN
 	1    3150 1000
 	1    0    0    -1
@@
 Wire Wire Line
 	9050 6050 9300 6050
+Wire Wire Line
+	2150 4250 2150 4750
+Wire Wire Line
+	2150 5050 2150 5500
+Wire Wire Line
+	850  4250 850  4750
+Wire Wire Line
+	850  5050 850  5500
+Text Label 4250 3050 2    50   ~ 0
+ITH
+Text Label 4250 3850 2    50   ~ 0
+VC
+Wire Wire Line
+	4550 3050 4250 3050
+Wire Wire Line
+	4550 3850 4250 3850
 $EndSCHEMATC

Commit message: Intermediate state.
Parts:
- removed C7: 200n, Capacitor_SMD:C_1812_4532Metric, symbol Device:C
- removed JP18: Top Side Current Shunt, Connector_PinHeader_2.54mm:PinHeader_1x02_P2.54mm_Vertical, symbol Device:Jumper_NC_Small
- removed JP19: Low Side Current Shunt, Connector_PinHeader_2.54mm:PinHeader_1x02_P2.54mm_Vertical, symbol Device:Jumper_NC_Small
- removed L1: 680n, footprints:INDPM7366X500N, symbol pspice:INDUCTOR
- removed R11, R12: 5m, footprints:CST0612-FC-R002E, symbol 2021-06-29_19-28-22:CST0612-FC-R002E
- removed U2, U3: SI7272DP-T1-GE3, footprints:SI7272DP-T1-GE3, symbol 2021-05-31_14-10-46:SI7272DP-T1-GE3
Other:
- moved on the sheet: C8, J3, JP20, Q1, R14, R15, R19

Commit message: Incorporated feedback into BCC and SCC - Fixed "unspecified" pin type warnings - Added correct test point symbols - Added thermal blockers - Added DRC parameters and fixed DRC issues - Adapted CubeSat STS1 PCB template to not violate DRC
Parts:
- J10, J11, J6, J7, J8, J9: symbol Connector:Conn_01x01_Male -> Connector:TestPoint
Changed lines of the file:
@@
 	10000 2250 10300 2250
 $Comp
-L Connector:Conn_01x01_Male J7
+L Connector:TestPoint J7
 U 1 1 6101A7BC
-P 7500 6350
-F 0 "J7" H 7608 6531 50  0000 C CNN
-F 1 "TG1" H 7608 6440 50  0000 C CNN
-F 2 "Connector_PinHeader_2.54mm:PinHeader_1x01_P2.54mm_Vertical" H 7500 6350 50  0001 C CNN
-F 3 "~" H 7500 6350 50  0001 C CNN
-	1    7500 6350
-	0    -1   -1   0
-$EndComp
-$Comp
-L Connector:Conn_01x01_Male J8
+P 7350 6050
+F 0 "J7" H 7250 6150 50  0000 C CNN
+F 1 "TG1" V 7350 6300 50  0000 C CNN
+F 2 "Connector_PinHeader_2.54mm:PinHeader_1x01_P2.54mm_Vertical" H 7350 6050 50  0001 C CNN
+F 3 "~" H 7350 6050 50  0001 C CNN
+	1    7350 6050
+	-1   0    0    1
+$EndComp
+$Comp
+L Connector:TestPoint J8
 U 1 1 610207BE
-P 7750 6350
-F 0 "J8" H 7858 6531 50  0000 C CNN
-F 1 "TG2" H 7858 6440 50  0000 C CNN
-F 2 "Connector_PinHeader_2.54mm:PinHeader_1x01_P2.54mm_Vertical" H 7750 6350 50  0001 C CNN
-F 3 "~" H 7750 6350 50  0001 C CNN
-	1    7750 6350
-	0    -1   -1   0
-$EndComp
-$Comp
-L Connector:Conn_01x01_Male J9
+P 7550 6050
+F 0 "J8" H 7450 6150 50  0000 C CNN
+F 1 "TG2" V 7550 6300 50  0000 C CNN
+F 2 "Connector_PinHeader_2.54mm:PinHeader_1x01_P2.54mm_Vertical" H 7550 6050 50  0001 C CNN
+F 3 "~" H 7550 6050 50  0001 C CNN
+	1    7550 6050
+	-1   0    0    1
+$EndComp
+$Comp
+L Connector:TestPoint J9
 U 1 1 61020D7E
-P 8000 6350
-F 0 "J9" H 8108 6531 50  0000 C CNN
-F 1 "BG1" H 8108 6440 50  0000 C CNN
-F 2 "Connector_PinHeader_2.54mm:PinHeader_1x01_P2.54mm_Vertical" H 8000 6350 50  0001 C CNN
-F 3 "~" H 8000 6350 50  0001 C CNN
-	1    8000 6350
-	0    -1   -1   0
-$EndComp
-$Comp
-L Connector:Conn_01x01_Male J10
+P 7750 6050
+F 0 "J9" H 7650 6150 50  0000 C CNN
+F 1 "BG1" V 7750 6300 50  0000 C CNN
+F 2 "Connector_PinHeader_2.54mm:PinHeader_1x01_P2.54mm_Vertical" H 7750 6050 50  0001 C CNN
+F 3 "~" H 7750 6050 50  0001 C CNN
+	1    7750 6050
+	-1   0    0    1
+$EndComp
+$Comp
+L Connector:TestPoint J10
 U 1 1 61020F9D
-P 8250 6350
-F 0 "J10" H 8358 6531 50  0000 C CNN
-F 1 "BG2" H 8358 6440 50  0000 C CNN
-F 2 "Connector_PinHeader_2.54mm:PinHeader_1x01_P2.54mm_Vertical" H 8250 6350 50  0001 C CNN
-F 3 "~" H 8250 6350 50  0001 C CNN
-	1    8250 6350
-	0    -1   -1   0
-$EndComp
-Text Label 7500 6150 1    50   ~ 0
+P 7950 6050
+F 0 "J10" H 7850 6150 50  0000 C CNN
+F 1 "BG2" V 7950 6300 50  0000 C CNN
+F 2 "Connector_PinHeader_2.54mm:PinHeader_1x01_P2.54mm_Vertical" H 7950 6050 50  0001 C CNN
+F 3 "~" H 7950 6050 50  0001 C CNN
+	1    7950 6050
+	-1   0    0    1
+$EndComp
+Text Label 7350 6050 1    50   ~ 0
 TG1
-Text Label 7750 6150 1    50   ~ 0
+Text Label 7550 6050 1    50   ~ 0
 TG2
-Text Label 8000 6150 1    50   ~ 0
+Text Label 7750 6050 1    50   ~ 0
 BG1
-Text Label 8250 6150 1    50   ~ 0
+Text Label 7950 6050 1    50   ~ 0
 BG2
-Text Label 8500 6150 1    50   ~ 0
+Text Label 8150 6050 1    50   ~ 0
 BGATE
 $Comp
-L Connector:Conn_01x01_Male J11
+L Connector:TestPoint J11
 U 1 1 61023037
-P 8500 6350
-F 0 "J11" H 8608 6531 50  0000 C CNN
-F 1 "BGATE" H 8608 6440 50  0000 C CNN
-F 2 "Connector_PinHeader_2.54mm:PinHeader_1x01_P2.54mm_Vertical" H 8500 6350 50  0001 C CNN
-F 3 "~" H 8500 6350 50  0001 C CNN
-	1    8500 6350
-	0    -1   -1   0
+P 8150 6050
+F 0 "J11" H 8050 6150 50  0000 C CNN
+F 1 "BGATE" V 8150 6350 50  0000 C CNN
+F 2 "Connector_PinHeader_2.54mm:PinHeader_1x01_P2.54mm_Vertical" H 8150 6050 50  0001 C CNN
+F 3 "~" H 8150 6050 50  0001 C CNN
+	1    8150 6050
+	-1   0    0    1
 $EndComp
 $Comp
@@
 Wire Wire Line
 	6250 6600 6250 6650
-Wire Wire Line
-	6600 6650 6550 6650
 Connection ~ 6250 6650
 Wire Wire Line
 	6250 6650 6250 6850
 $Comp
-L Connector:Conn_01x01_Male J6
+L Connector:TestPoint J6
 U 1 1 610C8A04
-P 6550 6850
-F 0 "J6" V 6650 6800 50  0000 R CNN
-F 1 "SHDN" V 6550 6800 50  0000 R CNN
-F 2 "Connector_PinHeader_2.54mm:PinHeader_1x01_P2.54mm_Vertical" H 6550 6850 50  0001 C CNN
-F 3 "~" H 6550 6850 50  0001 C CNN
-	1    6550 6850
-	0    -1   -1   0
-$EndComp
-Connection ~ 6550 6650
-Wire Wire Line
-	6550 6650 6250 6650
+P 7150 6050
+F 0 "J6" H 7100 6150 50  0000 R CNN
+F 1 "SHDN" V 7150 6450 50  0000 R CNN
+F 2 "Connector_PinHeader_2.54mm:PinHeader_1x01_P2.54mm_Vertical" H 7150 6050 50  0001 C CNN
+F 3 "~" H 7150 6050 50  0001 C CNN
+	1    7150 6050
+	-1   0    0    1
+$EndComp
 Wire Wire Line
 	10650 1650 10650 750
@@
 Wire Wire Line
 	7950 3150 7850 3150
+Wire Wire Line
+	6250 6650 6600 6650
+Text Label 7150 6050 1    50   ~ 0
+SHDN
 $EndSCHEMATC

Commit message: Changed footprints of some components.
Parts:
- D2, D3: value D_Schottky -> SD1206T040S1R0; footprint footprints:RB168MM-40TFTR -> Diode_SMD:D_1206_3216Metric
- R19: footprint footprints:CST0612-FC-R002E -> Resistor_SMD:R_1206_3216Metric; symbol 2021-06-29_19-28-22:CST0612-FC-R002E -> Device:R; Part Nr. (none) -> PCS1206DR0100ET
- R21: value 600k -> 1M
Connections:
- net Vout: now also JP20.2, R14.1, R19.2; no longer R19.3
- net at Q1.1, R19.1: now also JP20.1, R15.1
Changed lines of the file:
@@
 Vout
-Wire Wire Line
-	10650 2300 10650 2150
 Wire Wire Line
 	4550 2650 4250 2650
@@
 P 1600 2900
 F 0 "D2" V 1646 2820 50  0000 R CNN
-F 1 "D_Schottky" V 1555 2820 50  0000 R CNN
-F 2 "footprints:RB168MM-40TFTR" H 1600 2900 50  0001 C CNN
-F 3 "~" H 1600 2900 50  0001 C CNN
+F 1 "SD1206T040S1R0" V 1555 2820 50  0000 R CNN
+F 2 "Diode_SMD:D_1206_3216Metric" H 1600 2900 50  0001 C CNN
+F 3 "https://www.mouser.at/datasheet/2/40/schottky-776407.pdf" H 1600 2900 50  0001 C CNN
 	1    1600 2900
 	0    -1   -1   0
@@
 P 1600 3400
 F 0 "D3" V 1646 3320 50  0000 R CNN
-F 1 "D_Schottky" V 1555 3320 50  0000 R CNN
-F 2 "footprints:RB168MM-40TFTR" H 1600 3400 50  0001 C CNN
-F 3 "~" H 1600 3400 50  0001 C CNN
+F 1 "SD1206T040S1R0" V 1555 3320 50  0000 R CNN
+F 2 "Diode_SMD:D_1206_3216Metric" H 1600 3400 50  0001 C CNN
+F 3 "https://www.mouser.at/datasheet/2/40/schottky-776407.pdf" H 1600 3400 50  0001 C CNN
 	1    1600 3400
 	0    -1   -1   0
@@
 	3300 5550 3300 5350
 $Comp
-L 2021-06-29_19-28-22:CST0612-FC-R002E R?
+L Device:R R?
 U 1 1 6115AF39
-P 10600 2700
+P 10650 1850
 AR Path="/6115AF39" Ref="R?"  Part="1"
 AR Path="/60B53241/6115AF39" Ref="R19"  Part="1"
-F 0 "R19" H 11350 2550 50  0000 L CNN
-F 1 "10m" H 11350 2750 50  0000 L CNN
-F 2 "footprints:CST0612-FC-R002E" V 10530 2700 50  0001 C CNN
-F 3 "https://www.mouser.at/datasheet/2/54/cst0612-777607.pdf" H 10600 2700 50  0001 C CNN
-	1    10600 2700
-	0    1    -1   0
+F 0 "R19" H 10750 1750 50  0000 L CNN
+F 1 "10m" H 10750 1850 50  0000 L CNN
+F 2 "Resistor_SMD:R_1206_3216Metric" V 10580 1850 50  0001 C CNN
+F 3 "https://www.mouser.at/datasheet/2/303/res_pcs-1665423.pdf" H 10650 1850 50  0001 C CNN
+F 4 "PCS1206DR0100ET" H 10650 1850 50  0001 C CNN "Part Nr."
+	1    10650 1850
+	1    0    0    1
 $EndComp
 Text Label 2400 4000 0    50   ~ 0
@@
 U 1 1 60F4B388
 P 10300 1850
-F 0 "JP20" V 10350 2050 50  0000 R CNN
+F 0 "JP20" V 10350 2100 50  0000 R CNN
 F 1 "Battery Current" V 10250 2500 50  0000 R CNN
 F 2 "Connector_PinHeader_2.54mm:PinHeader_1x02_P2.54mm_Vertical" H 10300 1850 50  0001 C CNN
@@
 $EndComp
 Wire Wire Line
-	10450 1500 10450 1650
-Wire Wire Line
-	10450 2250 10450 2150
-Wire Wire Line
 	10300 1750 10300 1500
 Connection ~ 10300 1500
 Wire Wire Line
-	10300 1500 10450 1500
-Wire Wire Line
 	10300 1950 10300 2250
 Connection ~ 10300 2250
-Wire Wire Line
-	10300 2250 10450 2250
 Wire Wire Line
 	10000 1500 10300 1500
@@
 AR Path="/60B53241/610C89F6" Ref="R21"  Part="1"
 F 0 "R21" V 6597 5721 60  0000 R CNN
-F 1 "600k" V 6703 5721 60  0000 R CNN
+F 1 "1M" V 6703 5721 60  0000 R CNN
 F 2 "footprints:TS53YL 20K 20&percent_" H 6675 5365 60  0001 C CNN
 F 3 "" H 6250 5800 60  0000 C CNN
@@
 	-1   0    0    1
 $EndComp
-Wire Wire Line
-	10650 1650 10650 750
 $Sheet
 S 9300 5850 550  300
@@
 Text Label 7150 6050 1    50   ~ 0
 SHDN
+Wire Wire Line
+	10650 750  10650 1500
+Wire Wire Line
+	10650 2000 10650 2250
+Wire Wire Line
+	10300 1500 10650 1500
+Connection ~ 10650 1500
+Wire Wire Line
+	10650 1500 10650 1700
+Wire Wire Line
+	10300 2250 10650 2250
+Connection ~ 10650 2250
+Wire Wire Line
+	10650 2250 10650 2300
 $EndSCHEMATC
