File: STS1_EPS/STS1_EPS_PROTO_BCC_LTC4020/STS1_EPS_PROTO_BCC_LTC4020.kicad_pcb (KiCad board)
At the start: 2 copper layers, 85 x 85 mm, 96 parts, among them CON1 DISCO-CON1, CON11 DISCO-CON1, CON2 DISCO-CON2, CON21 DISCO-CON2, J1 1729267, J10 BG2, J11 BGATE, J2 Output, J3 Terminal BAT, J4 External NTC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

Commit message: Changed footprints of some components.
Parts:
- added U5: logo, footprints:STLogoTiny, F.Cu at (148.3, 53.9)
- D2, D3: value D_Schottky -> SD1206T040S1R0; footprint footprints:RB168MM-40TFTR -> Diode_SMD:D_1206_3216Metric
- R19: footprint footprints:CST0612-FC-R002E -> Resistor_SMD:R_1206_3216Metric
- R21: value 600k -> 1M
- moved D2 0.25 mm to (158.2, 78.0)
- moved D3 0.25 mm to (160.5, 78.0)
Connections:
- net /EPS Battery Charger/switch_bridge/BOTTOM_LEFT renamed Net-(C7-Pad2)
- JP20 pad 2: Net-(JP20-Pad2) -> /EPS Battery Charger/Vout
- Q1 pad 1: Net-(Q1-Pad1) -> Net-(JP20-Pad1)
- R14 pad 1: Net-(JP20-Pad2) -> /EPS Battery Charger/Vout
- R19 pad 1: Net-(Q1-Pad1) -> Net-(JP20-Pad1)
- R19 pad 2: Net-(JP20-Pad1) -> /EPS Battery Charger/Vout
Routing:
- net /EPS Battery Charger/Vout: track 50.3 -> 101.0 mm, vias 4 -> 5
- net Net-(JP20-Pad2): track 47.5 -> 0.00 mm, vias 1 -> 0
- net /EPS Battery Charger/BST1: track 31.6 -> 33.8 mm
- net Net-(JP20-Pad1): track 11.5 -> 13.2 mm
- net /EPS Battery Charger/SW1: track 51.1 -> 51.9 mm
- net /EPS Battery Charger/INTVCC: track 8.06 -> 7.50 mm
- added copper zone on F.Cu, net Net-(JP20-Pad1)
- removed copper zone on F.Cu, net Net-(Q1-Pad1)
